Commit message: initial commit

File: gym_pybullet_drones/assets/green_cylinder.urdf (robot description, URDF)
Before this commit: robot red_cylinder, 1 links, 0 joints
Links:
- link cylinder: geometry collision cylinder length=10 radius=0.5; visual cylinder length=10 radius=0.5

File: gym_pybullet_drones/assets/orange_cylinder.urdf (robot description, URDF)
Before this commit: robot red_cylinder, 1 links, 0 joints
Links:
- link cylinder: geometry collision cylinder length=10 radius=0.5; visual cylinder length=10 radius=0.5

File: gym_pybullet_drones/assets/red_cylinder.urdf (robot description, URDF)
Before this commit: robot red_cylinder, 1 links, 0 joints
Links:
- link cylinder: geometry collision cylinder length=10 radius=0.5; visual cylinder length=10 radius=0.5
